Commit message: testing

File: wamv_target.urdf (robot description, URDF)
Before this commit: robot WAM-V, 36 links, 35 joints
Links:
- removed link wamv/ball_shooter_base_link
- removed link wamv/ball_shooter_launcher_link
Joints:
- removed joint wamv/ball_shooter_base_joint
- removed joint wamv/ball_shooter_launcher_joint
