Commit message: fixed thruster error
No need to add the urdf argument now.

File: install/share/vrx_gazebo/models/wamv/tmp/model.urdf (robot description, URDF)
Before this commit: robot WAM-V, 36 links, 35 joints
Links:
- removed link wamv/far_left_camera_link
- removed link wamv/far_left_camera_link_optical
- removed link wamv/far_left_camera_post_arm_link
- removed link wamv/far_left_camera_post_link
- removed link wamv/stern_port1_engine_link
- removed link wamv/stern_port1_propeller_link
- removed link wamv/stern_port2_engine_link
- removed link wamv/stern_port2_propeller_link
- removed link wamv/stern_star1_engine_link
- removed link wamv/stern_star1_propeller_link
- removed link wamv/stern_star2_engine_link
- removed link wamv/stern_star2_propeller_link
- added link wamv/middle_right_camera_link, mass 0.3; collision box size=0.036 0.03 0.03; collision cylinder length=0.042 radius=0.015
- added link wamv/middle_right_camera_link_optical
- added link wamv/middle_right_camera_post_arm_link, mass 0.1; collision cylinder length=0.065 radius=0.008; visual mesh filename=package://vrx_gazebo/models/sensor_post/mesh/sensor_post_ar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
- added link wamv/middle_right_camera_post_link, mass 0.15885000000000002; collision cylinder length=0.17650000000000002 radius=0.0076; visual cylinder length=0.17650000000000002 radius=0.0076
- added link wamv/stern_port_engine_link, mass 15; collision box size=0.12 0.15 0.12; collision box size=0.2 0.15 0.83
- added link wamv/stern_port_propeller_link, mass 0.5; collision cylinder length=0.18 radius=0.24; visual mesh filename=package://wamv_description/models/propeller/mesh/propeller.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
- added link wamv/stern_star_engine_link, mass 15; collision box size=0.12 0.15 0.12; collision box size=0.2 0.15 0.83
- added link wamv/stern_star_propeller_link, mass 0.5; collision cylinder length=0.18 radius=0.24; visual mesh filename=package://wamv_description/models/propeller/mesh/propeller.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
Joints:
- removed joint wamv/base_to_far_left_camera_post_joint
- removed joint wamv/far_left_camera_post_arm_to_far_left_camera_joint
- removed joint wamv/far_left_camera_post_to_far_left_camera_post_arm_joint
- removed joint wamv/far_left_camera_to_far_left_camera_link_optical_joint
- removed joint wamv/stern_port1_chassis_engine_joint
- removed joint wamv/stern_port1_engine_propeller_joint
- removed joint wamv/stern_port2_chassis_engine_joint
- removed joint wamv/stern_port2_engine_propeller_joint
- removed joint wamv/stern_star1_chassis_engine_joint
- removed joint wamv/stern_star1_engine_propeller_joint
- removed joint wamv/stern_star2_chassis_engine_joint
- removed joint wamv/stern_star2_engine_propeller_joint
- added joint wamv/base_to_middle_right_camera_post_joint: type fixed, parent wamv/base_link, child wamv/middle_right_camera_post_link, origin xyz=0.5 -0.4 1.38475 rpy=0 0 -1.5707963267948966
- added joint wamv/middle_right_camera_post_arm_to_middle_right_camera_joint: type fixed, parent wamv/middle_right_camera_post_arm_link, child wamv/middle_right_camera_link, origin xyz=0.02 0 0.027 rpy=0 0.2617993877991494 0.0
- added joint wamv/middle_right_camera_post_to_middle_right_camera_post_arm_joint: type fixed, parent wamv/middle_right_camera_post_link, child wamv/middle_right_camera_post_arm_link, origin xyz=0.03 0 0.08825000000000008 rpy=0 0 0
- added joint wamv/middle_right_camera_to_middle_right_camera_link_optical_joint: type fixed, parent wamv/middle_right_camera_link, child wamv/middle_right_camera_link_optical, origin xyz=0 0 0 rpy=-1.5707963267948966 0 -1.5707963267948966
- added joint wamv/stern_port_chassis_engine_joint: type revolute, parent wamv/base_link, child wamv/stern_port_engine_link, origin xyz=-1.05 0.8 0.318237 rpy=0.0 0.0 0.0, axis 0 0 1, limit lower=-3.141592653589793 upper=3.141592653589793 effort=10 velocity=10
- added joint wamv/stern_port_engine_propeller_joint: type continuous, parent wamv/stern_port_engine_link, child wamv/stern_port_propeller_link, origin xyz=-0.278156 0 -0.509371 rpy=0 0 0, axis 1 0 0, limit effort=100 velocity=100
- added joint wamv/stern_star_chassis_engine_joint: type revolute, parent wamv/base_link, child wamv/stern_star_engine_link, origin xyz=-1.05 -0.8 0.318237 rpy=0.0 0.0 0.0, axis 0 0 1, limit lower=-3.141592653589793 upper=3.141592653589793 effort=10 velocity=10
- added joint wamv/stern_star_engine_propeller_joint: type continuous, parent wamv/stern_star_engine_link, child wamv/stern_star_propeller_link, origin xyz=-0.278156 0 -0.509371 rpy=0 0 0, axis 1 0 0, limit effort=100 velocity=100
- joint wamv/ball_shooter_base_joint: origin xyz=0.55 -0.3 1.3 rpy=0 0 0.0 -> xyz=0.54 0.3 1.296 rpy=0 0 0
- joint wamv/ball_shooter_launcher_joint: origin xyz=-0.0204 0 0.107877 rpy=0 -0.3490658503988659 0 -> xyz=-0.0204 0 0.107877 rpy=0 -1.04 0
- joint wamv/base_to_front_left_camera_post_joint: origin xyz=0.7 0.1 1.38475 rpy=0 0 0.0 -> xyz=0.7 0.1 1.38475 rpy=0 0 0
- joint wamv/base_to_front_right_camera_post_joint: origin xyz=0.7 -0.1 1.38475 rpy=0 0 0.0 -> xyz=0.7 -0.1 1.38475 rpy=0 0 0
- joint wamv/base_to_lidar_wamv_post_joint: origin xyz=0.6299999999999999 0.0 1.52325 rpy=0 0 0.0 -> xyz=0.6299999999999999 0.0 1.52325 rpy=0 0 0
- joint wamv/bow_port_chassis_engine_joint: type fixed -> revolute
- joint wamv/bow_star_chassis_engine_joint: type fixed -> revolute
- joint wamv/front_left_camera_post_arm_to_front_left_camera_joint: origin xyz=0.02 0 0.027 rpy=0.0 0.2617993877991494 0.0 -> xyz=0.02 0 0.027 rpy=0 0.2617993877991494 0
- joint wamv/front_right_camera_post_arm_to_front_right_camera_joint: origin xyz=0.02 0 0.027 rpy=0.0 0.2617993877991494 0.0 -> xyz=0.02 0 0.027 rpy=0 0.2617993877991494 0
- joint wamv/gps_wamv_joint: origin xyz=-0.85 0.0 1.3 rpy=0.0 0.0 0.0 -> xyz=-0.85 0 1.3 rpy=0 0 0
- joint wamv/imu_wamv_joint: origin xyz=0.3 -0.2 1.3 rpy=0.0 0.0 0.0 -> xyz=0.3 -0.2 1.3 rpy=0 0 0
- joint wamv/lidar_wamv_post_arm_to_lidar_wamv_joint: origin xyz=0.04 0 0.05 rpy=0.0 0.13962634015954636 0.0 -> xyz=0.04 0 0.05 rpy=0 0 0

File: install/share/wamv_gazebo/urdf/thruster_layouts/wamv_x_thrusters.xacro (robot description, xacro)
@@ -2,12 +2,12 @@
 <robot xmlns:xacro="http://ros.org/wiki/xacro">
   <xacro:include filename="$(find wamv_description)/urdf/thrusters/engine.xacro" />
-  <xacro:engine prefix="left_rear" position="-2.373776 1.027135 0.318237"  orientation="0.0 0.0 0.785"/>
-  <xacro:engine prefix="right_rear" position="-2.373776 -1.027135 0.318237" orientation="0.0 0.0 -0.785"/>
-  <xacro:engine prefix="left_front" position="1.6 0.7  0.25" orientation="0.0 0.0 -0.785"/>
-  <xacro:engine prefix="right_front" position="1.6 -0.7 0.25" orientation="0.0 0.0 +0.785"/>
+  <xacro:engine prefix="stern_port" position="-1.05 0.8 0.318237"  orientation="0.0 0.0 0.0"/>
+  <xacro:engine prefix="stern_star" position="-1.05 -0.8 0.318237" orientation="0.0 0.0 0.0"/>
+  <xacro:engine prefix="bow_port" position="1.2 0.9 0.318237" orientation="0.0 0.0 1.57"/>
+  <xacro:engine prefix="bow_star" position="1.2 -0.9 0.318237" orientation="0.0 0.0 -1.57"/>
   <xacro:include filename="$(find wamv_gazebo)/urdf/thruster_layouts/wamv_gazebo_thruster_config.xacro" />
-  <xacro:wamv_gazebo_thruster_config name="left_rear" />
-  <xacro:wamv_gazebo_thruster_config name="right_rear" />
-  <xacro:wamv_gazebo_thruster_config name="left_front" />
-  <xacro:wamv_gazebo_thruster_config name="right_front" />
+  <xacro:wamv_gazebo_thruster_config name="stern_port" />
+  <xacro:wamv_gazebo_thruster_config name="stern_star" />
+  <xacro:wamv_gazebo_thruster_config name="bow_port" />
+  <xacro:wamv_gazebo_thruster_config name="bow_star" />
 </robot>

File: install/share/wamv_gazebo/urdf/wamv_gazebo.urdf.xacro (robot description, xacro)
@@ -49,5 +49,5 @@
     <!-- Default WAM-V with two aft thrusters -->
     <xacro:if value="${thruster_conf == 'H'}">
-       <xacro:wamv_gazebo thruster_layout="$(find wamv_gazebo)/urdf/thruster_layouts/wamv_aft_thrusters.xacro"/>
+       <xacro:wamv_gazebo thruster_layout="$(find wamv_gazebo)/urdf/thruster_layouts/wamv_x_thrusters.xacro"/>
     </xacro:if>
     <!-- WAMV with "T" thruster configuration -->

Commit message: added controller.py

File: install/share/vrx_gazebo/models/wamv/tmp/model.urdf (robot description, URDF)
Before this commit: robot WAM-V, 32 links, 31 joints
Joints:
- joint wamv/bow_port_chassis_engine_joint: origin xyz=1.2 0.9 0.318237 rpy=0.0 0.0 1.57 -> xyz=1.2 0.5 0.318237 rpy=0.0 0.0 -1.57
- joint wamv/bow_star_chassis_engine_joint: origin xyz=1.2 -0.9 0.318237 rpy=0.0 0.0 -1.57 -> xyz=1.2 -0.5 0.318237 rpy=0.0 0.0 1.57

File: install/share/wamv_gazebo/urdf/thruster_layouts/wamv_x_thrusters.xacro (robot description, xacro)
@@ -4,6 +4,6 @@
   <xacro:engine prefix="stern_port" position="-1.05 0.8 0.318237"  orientation="0.0 0.0 0.0"/>
   <xacro:engine prefix="stern_star" position="-1.05 -0.8 0.318237" orientation="0.0 0.0 0.0"/>
-  <xacro:engine prefix="bow_port" position="1.2 0.9 0.318237" orientation="0.0 0.0 1.57"/>
-  <xacro:engine prefix="bow_star" position="1.2 -0.9 0.318237" orientation="0.0 0.0 -1.57"/>
+  <xacro:engine prefix="bow_port" position="1.2 0.5 0.318237" orientation="0.0 0.0 -1.57"/>
+  <xacro:engine prefix="bow_star" position="1.2 -0.5 0.318237" orientation="0.0 0.0 1.57"/>
   <xacro:include filename="$(find wamv_gazebo)/urdf/thruster_layouts/wamv_gazebo_thruster_config.xacro" />
   <xacro:wamv_gazebo_thruster_config name="stern_port" />
